File: esp32s3-wroom-learnpcb.kicad_sch (KiCad schematic)
At the start: 0 parts

Commit message: POC(schem): add ESP32-S3-WROOM-1 symbol
Other:
- added sheet POC (poc.kicad_sch)
Changed lines of the file:
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@@
 	(generator_version "9.0")
 	(paper "A4")
+	(sheet
+		(at 53.34 57.15)
+		(size 12.7 22.86)
+		(exclude_from_sim no)
+		(in_bom yes)
+		(on_board yes)
+		(dnp no)
+		(fields_autoplaced yes)
+		(stroke
+			(width 0.1524)
+			(type solid)
+		)
+		(fill
+			(color 0 0 0 0.0000)
+		)
+		(property "Sheetname" "POC"
+			(at 53.34 56.4384 0)
+			(effects
+				(font
+					(size 1.27 1.27)
+				)
+				(justify left bottom)
+			)
+		)
+		(property "Sheetfile" "poc.kicad_sch"
+			(at 53.34 80.5946 0)
+			(effects
+				(font
+					(size 1.27 1.27)
+				)
+				(justify left top)
+			)
+		)
+		(instances
+			(project "esp32s3-wroom-learnpcb"
+				(path "/93de29fe-314e-498a-b627-688058496610"
+					(page "2")
+				)
+			)
+		)
+	)
 	(sheet_instances
 		(path "/"
